File: PCB/zepto_duo_terminal.kicad_pcb (KiCad board)
At the start: 2 copper layers, 400 x 120 mm, 179 parts, among them J1 VGA, J5 Conn_01x04, J7 Conn_01x03, J8 Conn_01x03

Commit message: Minor changes to case and PCB
Routing:
- net COL_3: track 449.3 -> 444.7 mm, vias 3 -> 4
- net GND: vias 86 -> 92
Changed lines of the file:
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@@
+	)
+	(via
+		(at 345.998 282.667)
+		(size 0.6)
+		(drill 0.3)
+		(layers "F.Cu" "B.Cu")
+		(free yes)
+		(net 2)
+	)
+	(via
+		(at 296.722 280.127)
+		(size 0.6)
+		(drill 0.3)
+		(layers "F.Cu" "B.Cu")
+		(free yes)
+		(net 2)
 	)
 	(via
@@
 	)
 	(via
+		(at 339.902 279.111)
+		(size 0.6)
+		(drill 0.3)
+		(layers "F.Cu" "B.Cu")
+		(free yes)
+		(net 2)
+	)
+	(via
 		(at 420 280)
 		(size 0.6)
@@
 	)
 	(via
+		(at 326.186 270.983)
+		(size 0.6)
+		(drill 0.3)
+		(layers "F.Cu" "B.Cu")
+		(free yes)
+		(net 2)
+	)
+	(via
 		(at 459 226)
 		(size 0.6)
@@
 	)
 	(via
+		(at 345.49 263.871)
+		(size 0.6)
+		(drill 0.3)
+		(layers "F.Cu" "B.Cu")
+		(free yes)
+		(net 2)
+	)
+	(via
 		(at 475 243)
 		(size 0.6)
@@
 	(via
 		(at 427 220)
+		(size 0.6)
+		(drill 0.3)
+		(layers "F.Cu" "B.Cu")
+		(free yes)
+		(net 2)
+	)
+	(via
+		(at 348.538 271.491)
 		(size 0.6)
 		(drill 0.3)
@@
 	)
 	(segment
+		(start 228.65 260.95)
+		(end 228.65 267.65)
+		(width 0.2)
+		(layer "F.Cu")
+		(net 14)
+	)
+	(segment
+		(start 270.0974 274.9255)
+		(end 272.1719 277)
+		(width 0.2)
+		(layer "F.Cu")
+		(net 14)
+	)
+	(segment
 		(start 400 228.814816)
 		(end 400 260.85)
@@
 	)
 	(segment
+		(start 272.1719 277)
+		(end 339 277)
+		(width 0.2)
+		(layer "F.Cu")
+		(net 14)
+	)
+	(segment
 		(start 339 277)
 		(end 394 277)
@@
 	)
 	(segment
-		(start 228.65 260.95)
-		(end 228.65 267.65)
+		(start 228.65 267.65)
+		(end 235.9255 274.9255)
 		(width 0.2)
 		(layer "F.Cu")
@@
 	)
 	(segment
-		(start 238 277)
-		(end 339 277)
-		(width 0.2)
-		(layer "F.Cu")
-		(net 14)
-	)
-	(segment
 		(start 228.65 203.8)
 		(end 228.65 260.95)
@@
 	)
 	(segment
-		(start 228.65 267.65)
-		(end 238 277)
-		(width 0.2)
-		(layer "F.Cu")
-		(net 14)
-	)
-	(segment
 		(start 394 277)
 		(end 400.1 270.9)
@@
 	)
 	(segment
+		(start 235.9255 274.9255)
+		(end 270.0974 274.9255)
+		(width 0.2)
+		(layer "F.Cu")
+		(net 14)
+	)
+	(segment
 		(start 423.7 201.3)
 		(end 429.22 201.3)
@@
 	)
 	(segment
+		(start 304.85 280)
+		(end 319 280)
+		(width 0.2)
+		(layer "F.Cu")
+		(net 19)
+	)
+	(segment
 		(start 304.1661 198.599)
 		(end 304.401 198.599)
@@
 		(net 19)
 	)
+	(segment
+		(start 319 280)
+		(end 319.1005 280.1005)
+		(width 0.2)
+		(layer "F.Cu")
+		(net 19)
+	)
 	(via
 		(at 361 275)
@@
 	(via
 		(at 369.58 196.22)
+		(size 0.6)
+		(drill 0.3)
+		(layers "F.Cu" "B.Cu")
+		(net 19)
+	)
+	(via
+		(at 319.1005 280.1005)
 		(size 0.6)
 		(drill 0.3)
@@
 	)
 	(segment
-		(start 319 280)
-		(end 300.0875 280)
-		(width 0.2)
-		(layer "B.Cu")
-		(net 19)
-	)
-	(segment
 		(start 321 196)
 		(end 321.22 196.22)
@@
 	)
 	(segment
+		(start 319.1005 280.1005)
+		(end 319 280)
+		(width 0.2)
+		(layer "B.Cu")
+		(net 19)
+	)
+	(segment
 		(start 328 279)
 		(end 325 282)
@@
 	(segment
 		(start 321 282)
-		(end 319 280)
+		(end 319.1005 280.1005)
 		(width 0.2)
 		(layer "B.Cu")
@@
 	)
 	(segment
-		(start 253.599 276.599)
+		(start 270.2635 274.5245)
+		(end 272.338 276.599)
+		(width 0.2)
+		(layer "F.Cu")
+		(net 20)
+	)
+	(segment
+		(start 272.338 276.599)
 		(end 363.401 276.599)
 		(width 0.2)
@@
 	)
 	(segment
+		(start 251.5245 274.5245)
+		(end 270.2635 274.5245)
+		(width 0.2)
+		(layer "F.Cu")
+		(net 20)
+	)
+	(segment
 		(start 395.599 277.401)
 		(end 404 269)
@@
 	(segment
 		(start 247.7 270.7)
-		(end 253.599 276.599)
-		(width 0.2)
-		(layer "F.Cu")
+		(end 251.5245 274.5245)
+		(width 0.2)
+		(layer "F.Cu")
